File: H1AR20/Design/H1AR20.sch (EAGLE design)
At the start: 42 parts, among them J1 67503-1020, P1 HEXABIT_17.32_NO_P3, U1 STM32F091CBU6, U2 LM3940IMP-3.3, U3 FT230XQ-R, X1 XTALL_CSTCE8M00G52

Commit message: - renamed res and cap to match the original Circuitmaker  design - fixed BOM file according to changes
Parts:
- C1: value 10nF -> 100nF; CAPACITANCE 10nF -> 100nF; MPN C0603C103K5RACTU -> C0603C104K8RACTU; OCTOPART_URL https://octopart.com/c0603c103k5ractu-kemet-133094?r=sp&s=R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 -> https://octopart.com/c0603c104k8ractu-kemet-145075?r=sp&s=9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; VOLTAGE_RATING 50V -> 10V
- C10: value 1uF -> 4.7uF; CAPACITANCE 1.00 µF -> 4.7 µF; MFN AVX -> Panasonic; MPN TAJR105M016RNJ -> 10TPU4R7MSI; OCTOPART_URL http://octopart.com/tajr105m016rnj-avx-1188552 -> https://octopart.com/10tpu4r7msi-panasonic-29487748; VOLTAGE_RATING 16.0 V -> 10.0 V
- C11: value 100uF -> 100nF; device Hexabitz:C-3225TDK_C3225X5R0J107M250AC_0_0 -> Hexabitz:C-0603; CAPACITANCE (none) -> 100 nF; MFN (none) -> AVX; MPN (none) -> 0603YC104K4T2A; OCTOPART_URL (none) -> https://octopart.com/0603yc104k4t2a-avx+interconnect+%2F+el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; TOLERANCE (none) -> ±10%; VOLTAGE_RATING (none) -> 16.0 V
- C12: value 47pF -> 100nF; CAPACITANCE 47 pF -> 100 nF; MPN 06035A470JAT2A -> 0603YC104K4T2A; OCTOPART_URL https://octopart.com/c3225x5r0j107m250ac-tdk-25947844?r=spc# -> https://octopart.com/0603yc104k4t2a-avx+interconnect+%2F+el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; TOLERANCE ±5% -> ±10%; VOLTAGE_RATING 50.0 V -> 16.0 V
- C13: OCTOPART_URL https://octopart.com/06035a470jat2a-avx+interconnect+%2F+el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 -> https://octopart.com/c3225x5r0j107m250ac-tdk-25947844?r=spc#
- C14: value 100nF -> 47pF; CAPACITANCE 100 nF -> 47 pF; MPN 0603YC104K4T2A -> 06035A470JAT2A; OCTOPART_URL https://octopart.com/0603yc104k4t2a-avx+interconnect+%2F+el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 -> https://octopart.com/06035a470jat2a-avx+interconnect+%2F+el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; TOLERANCE ±10% -> ±5%; VOLTAGE_RATING 16.0 V -> 50.0 V
- C16: value 100nF -> 100uF; device Hexabitz:C-0603 -> Hexabitz:C-3225TDK_C3225X5R0J107M250AC_0_0; CAPACITANCE 100 nF -> (none); MFN AVX -> (none); MPN 0603YC104K4T2A -> (none); OCTOPART_URL https://octopart.com/0603yc104k4t2a-avx+interconnect+%2F+el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 -> (none); TOLERANCE ±10% -> (none); VOLTAGE_RATING 16.0 V -> (none)
- C17: value 4.7uF -> 1uF; CAPACITANCE 4.7 µF -> 1.00 µF; MFN Panasonic -> AVX; MPN 10TPU4R7MSI -> TAJR105M016RNJ; OCTOPART_URL https://octopart.com/10tpu4r7msi-panasonic-29487748 -> http://octopart.com/tajr105m016rnj-avx-1188552; VOLTAGE_RATING 10.0 V -> 16.0 V
- C3: value 100nF -> 4.7uF; device Hexabitz:C-0603 -> Hexabitz:C-0805-POL; CAPACITANCE 100nF -> 4.7uF; MFN KEMET -> Murata; MPN C0603C104K8RACTU -> GRM21BC81E475KA12L; OCTOPART_URL https://octopart.com/c0603c104k8ractu-kemet-145075?r=sp&s=9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 -> https://octopart.com/grm21bc81e475ka12l-murata-10331911?r=s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; VOLTAGE_RATING 10V -> 25V
- C5: value 100nF -> 10nF; CAPACITANCE 100nF -> 10nF; MPN C0603C104K8RACTU -> C0603C103K5RACTU; OCTOPART_URL https://octopart.com/c0603c104k8ractu-kemet-145075?r=sp&s=9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 -> https://octopart.com/c0603c103k5ractu-kemet-133094?r=sp&s=R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; VOLTAGE_RATING 10 -> 50V
- C7: value 4.7uF -> 100nF; device Hexabitz:C-0805-POL -> Hexabitz:C-0603; CAPACITANCE 4.7uF -> 100nF; MFN Murata -> KEMET; MPN GRM21BC81E475KA12L -> C0603C104K8RACTU; OCTOPART_URL https://octopart.com/grm21bc81e475ka12l-murata-10331911?r=s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 -> https://octopart.com/c0603c104k8ractu-kemet-145075?r=sp&s=9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; VOLTAGE_RATING 25V -> 10
- R2: value 0.0R -> 10.0K; MFN Yageo -> Vishay; MPN RC0603JR-070RL -> CRCW060310K0JNEB; OCTOPART_URL https://octopart.com/rc0603jr-070rl-yageo-1241539?r=sp&s=X2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 -> https://octopart.com/crcw060310k0jneb-vishay+dale-46603268; RESISTANCE 0.0 Ohm -> 10.0K Ohm; TOLERANCE (none) -> 5%
- R3: value 10.0K -> 0.0R; MFN Vishay -> Yageo; MPN CRCW060310K0JNEB -> RC0603JR-070RL; OCTOPART_URL https://octopart.com/crcw060310k0jneb-vishay+dale-46603268 -> https://octopart.com/rc0603jr-070rl-yageo-1241539?r=sp&s=X2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; RESISTANCE 10.0K Ohm -> 0.0 Ohm; TOLERANCE 5% -> (none)
- R4: value 4.7kΩ -> 27.0Ω; MPN CRCW06034K70FKEA -> CRCW060327R0FKEA; OCTOPART_URL http://octopart.com/crcw06034k70fkea-vishay-39455708 -> https://octopart.com/crcw060327r0fkea-vishay-39833156; RESISTANCE 4.7 kΩ -> 27.0 Ω
- R5: value 10kΩ -> 27.0Ω; MPN CRCW060310K0JNEB -> CRCW060327R0FKEA; OCTOPART_URL https://octopart.com/crcw060310k0jneb-vishay+dale-46603268 -> https://octopart.com/crcw060327r0fkea-vishay-39833156; RESISTANCE 10.0 kΩ -> 27.0 Ω; TOLERANCE ±5% -> ±1%
- R6: value 27.0Ω -> 39.0Ω; MFN Vishay -> Panasonic; MPN CRCW060327R0FKEA -> ERJ-3GEYJ390V; OCTOPART_URL https://octopart.com/crcw060327r0fkea-vishay-39833156 -> https://octopart.com/erj-3geyj390v-panasonic-55422095; RESISTANCE 27.0 Ω -> 39.0 Ω; TOLERANCE ±1% -> ±5%
- R7: value 27.0Ω -> 270.0Ω; MFN Vishay -> Panasonic; MPN CRCW060327R0FKEA -> ERJ-3GEYJ271V; OCTOPART_URL https://octopart.com/crcw060327r0fkea-vishay-39833156 -> https://octopart.com/erj-3geyj271v-panasonic-55560546; RESISTANCE 27.0 Ω -> 270.0 Ω; TOLERANCE ±1% -> ±5%
- R8: value 270.0Ω -> 4.7kΩ; MFN Panasonic -> Vishay; MPN ERJ-3GEYJ271V -> CRCW06034K70FKEA; OCTOPART_URL https://octopart.com/erj-3geyj271v-panasonic-55560546 -> http://octopart.com/crcw06034k70fkea-vishay-39455708; RESISTANCE 270.0 Ω -> 4.7 kΩ; TOLERANCE ±5% -> ±1%
- R9: value 39.0Ω -> 10kΩ; MFN Panasonic -> Vishay; MPN ERJ-3GEYJ390V -> CRCW060310K0JNEB; OCTOPART_URL https://octopart.com/erj-3geyj390v-panasonic-55422095 -> https://octopart.com/crcw060310k0jneb-vishay+dale-46603268; RESISTANCE 39.0 Ω -> 10.0 kΩ
Connections:
- net B1: now also R2.2; no longer R3.2
- net GND: now also C1.2, C11.2, C16.1, C3.-, C7.2, R9.1; no longer C11.1, C16.2, C3.2, C5.2, C7.-, R5.1
- net N$11: now also C17.+; no longer C10.+
- net N$12: now also R5.2; no longer R7.2
- net N$13: now also R4.2; no longer R6.2
- net N$14: now also R7.1; no longer R8.1
- net N$15: now also R6.1; no longer R9.1
- net N$16: now also R7.2; no longer R8.2
- net N$17: now also R6.2; no longer R9.2
- net N$18: now also R8.2; no longer R4.2
- net N$2: now also C14.1, R4.1; no longer C13.1, R6.1
- net N$3: now also C13.1, R5.1; no longer C12.1, R7.1
- net R1: now also C1.1; no longer C8.1
- net VBUS_SENSE: now also R8.1, R9.2; no longer R4.1, R5.2
- net VDD: now also C10.+, C11.1, C12.1, C16.2, C3.+, C7.1, C8.1; no longer C11.2, C14.1, C16.1, C17.+, C3.1, C5.1, C7.+
- net VDDA: now also C5.1; no longer C1.1
- net VSSA: now also C5.2, R3.2; no longer C1.2, R2.2
Other:
- moved on the sheet: C1, C10, C12, C13, C14, C15, C17, C4, C5, C6, C8, R2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

Commit message: replaced labels "USART" with "UART"
Connections:
- net USART1_CTS renamed UART1_CTS
- net USART1_RTS renamed UART1_RTS
- net USART1_RX renamed UART1_RX
- net USART1_TX renamed UART1_TX
- net USART2_RX renamed UART2_RX
- net USART2_TX renamed UART2_TX
- net USART3_RX renamed UART3_RX
- net USART3_TX renamed UART3_TX
- net USART4_RX renamed UART4_RX
- net USART4_TX renamed UART4_TX
- net USART5_RX renamed UART5_RX
- net USART5_TX renamed UART5_TX
- net USART6_RX renamed UART6_RX
- net USART6_TX renamed UART6_TX
Other:
- moved on the sheet: C, D
Changed lines of the file:
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@@
 <setting verticaltext="up"/>
 </settings>
-<grid distance="0.1" unitdist="inch" unit="inch" style="lines" multiple="1" display="yes" altdistance="0.01" altunitdist="inch" altunit="inch"/>
+<grid distance="50" unitdist="mil" unit="mil" style="lines" multiple="1" display="yes" altdistance="0.01" altunitdist="inch" altunit="inch"/>
 <layers>
 <layer number="1" name="Top" color="4" fill="1" visible="no" active="no"/>
@@
 <attribute name="VALUE" x="182.753" y="53.975" size="1.778" layer="96"/>
 </instance>
-<instance part="D" gate="G$1" x="115.57" y="144.78" smashed="yes" rot="R180">
-<attribute name="NAME" x="111.76" y="144.78" size="1.27" layer="95" rot="R180"/>
-<attribute name="VALUE" x="116.84" y="148.59" size="1.27" layer="96" rot="R180"/>
-</instance>
-<instance part="C" gate="G$1" x="115.57" y="140.97" smashed="yes" rot="R180">
-<attribute name="NAME" x="111.76" y="140.97" size="1.27" layer="95" rot="R180"/>
-<attribute name="VALUE" x="116.84" y="138.43" size="1.27" layer="96" rot="R180"/>
+<instance part="D" gate="G$1" x="115.57" y="132.08" smashed="yes" rot="R180">
+<attribute name="NAME" x="111.76" y="132.08" size="1.27" layer="95" rot="R180"/>
+<attribute name="VALUE" x="116.84" y="135.89" size="1.27" layer="96" rot="R180"/>
+</instance>
+<instance part="C" gate="G$1" x="115.57" y="128.27" smashed="yes" rot="R180">
+<attribute name="NAME" x="111.76" y="128.27" size="1.27" layer="95" rot="R180"/>
+<attribute name="VALUE" x="116.84" y="125.73" size="1.27" layer="96" rot="R180"/>
 </instance>
 <instance part="B" gate="G$1" x="252.73" y="129.54" smashed="yes">
@@
 </segment>
 </net>
-<net name="USART1_TX" class="0">
+<net name="UART1_TX" class="0">
 <segment>
-<wire x1="135.89" y1="154.94" x2="119.38" y2="154.94" width="0.1524" layer="91"/>
-<label x="119.38" y="154.94" size="1.778" layer="95"/>
+<wire x1="135.89" y1="154.94" x2="129.54" y2="154.94" width="0.1524" layer="91"/>
 <pinref part="U1" gate="G$1" pin="PA9"/>
+<label x="129.54" y="154.94" size="1.778" layer="95" rot="R180" xref="yes"/>
 </segment>
 </net>
-<net name="USART1_RX" class="0">
+<net name="UART1_RX" class="0">
 <segment>
-<wire x1="135.89" y1="152.4" x2="119.38" y2="152.4" width="0.1524" layer="91"/>
-<label x="119.38" y="152.4" size="1.778" layer="95"/>
+<wire x1="135.89" y1="152.4" x2="123.19" y2="152.4" width="0.1524" layer="91"/>
 <pinref part="U1" gate="G$1" pin="PA10"/>
+<wire x1="123.19" y1="152.4" x2="123.19" y2="149.86" width="0.1524" layer="91"/>
+<wire x1="123.19" y1="149.86" x2="119.38" y2="149.86" width="0.1524" layer="91"/>
+<label x="119.38" y="149.86" size="1.778" layer="95" rot="R180" xref="yes"/>
 </segment>
 </net>
@@
 </segment>
 </net>
-<net name="N$7" class="0">
-<segment>
-<pinref part="U1" gate="G$1" pin="PA13"/>
-<pinref part="D" gate="G$1" pin="P$1"/>
-<wire x1="135.89" y1="144.78" x2="118.11" y2="144.78" width="0.1524" layer="91"/>
-</segment>
-</net>
 <net name="N$9" class="0">
 <segment>
 <pinref part="U1" gate="G$1" pin="PA14"/>
-<wire x1="135.89" y1="142.24" x2="120.65" y2="142.24" width="0.1524" layer="91"/>
-<wire x1="120.65" y1="142.24" x2="120.65" y2="140.97" width="0.1524" layer="91"/>
+<wire x1="135.89" y1="142.24" x2="133.35" y2="142.24" width="0.1524" layer="91"/>
+<wire x1="133.35" y1="142.24" x2="133.35" y2="128.27" width="0.1524" layer="91"/>
 <pinref part="C" gate="G$1" pin="P$1"/>
-<wire x1="120.65" y1="140.97" x2="118.11" y2="140.97" width="0.1524" layer="91"/>
+<wire x1="133.35" y1="128.27" x2="118.11" y2="128.27" width="0.1524" layer="91"/>
 </segment>
 </net>
-<net name="USART2_TX" class="0">
+<net name="UART2_TX" class="0">
 <segment>
 <pinref part="P1" gate="G$1" pin="SU1"/>
@@
 </segment>
 </net>
-<net name="USART6_TX" class="0">
+<net name="UART6_TX" class="0">
 <segment>
 <pinref part="P1" gate="G$1" pin="SU2"/>
@@
 </segment>
 </net>
-<net name="USART3_TX" class="0">
+<net name="UART3_TX" class="0">
 <segment>
 <pinref part="P1" gate="G$1" pin="SU4"/>
@@
 </segment>
 </net>
-<net name="USART4_TX" class="0">
+<net name="UART4_TX" class="0">
 <segment>
 <pinref part="P1" gate="G$1" pin="SU5"/>
@@
 </segment>
 </net>
-<net name="USART5_TX" class="0">
+<net name="UART5_TX" class="0">
 <segment>
 <pinref part="P1" gate="G$1" pin="SU6"/>
@@
 </segment>
 </net>
-<net name="USART2_RX" class="0">
+<net name="UART2_RX" class="0">
 <segment>
 <pinref part="P1" gate="G$1" pin="SD1"/>
@@
 </segment>
 </net>
-<net name="USART6_RX" class="0">
+<net name="UART6_RX" class="0">
 <segment>
 <pinref part="P1" gate="G$1" pin="SD2"/>
@@
 </segment>
 </net>
-<net name="USART3_RX" class="0">
+<net name="UART3_RX" class="0">
 <segment>
 <pinref part="P1" gate="G$1" pin="SD4"/>
@@
 </segment>
 </net>
-<net name="USART4_RX" class="0">
+<net name="UART4_RX" class="0">
 <segment>
 <pinref part="P1" gate="G$1" pin="SD5"/>
@@
 </segment>
 </net>
-<net name="USART5_RX" class="0">
+<net name="UART5_RX" class="0">
 <segment>
 <pinref part="P1" gate="G$1" pin="SD6"/>
@@
 </segment>
 </net>
-<net name="USART1_CTS" class="0">
+<net name="UART1_CTS" class="0">
 <segment>
 <pinref part="U1" gate="G$1" pin="PA11"/>
-<wire x1="135.89" y1="149.86" x2="119.38" y2="149.86" width="0.1524" layer="91"/>
-<label x="119.38" y="149.86" size="1.778" layer="95"/>
+<wire x1="135.89" y1="149.86" x2="125.73" y2="149.86" width="0.1524" layer="91"/>
+<wire x1="125.73" y1="149.86" x2="125.73" y2="144.78" width="0.1524" layer="91"/>
+<wire x1="125.73" y1="144.78" x2="119.38" y2="144.78" width="0.1524" layer="91"/>
+<label x="119.38" y="144.78" size="1.778" layer="95" rot="R180" xref="yes"/>
 </segment>
 </net>
-<net name="USART1_RTS" class="0">
+<net name="UART1_RTS" class="0">
 <segment>
 <pinref part="U1" gate="G$1" pin="PA12"/>
-<wire x1="135.89" y1="147.32" x2="119.38" y2="147.32" width="0.1524" layer="91"/>
-<label x="119.38" y="147.32" size="1.778" layer="95"/>
+<wire x1="135.89" y1="147.32" x2="128.27" y2="147.32" width="0.1524" layer="91"/>
+<wire x1="128.27" y1="147.32" x2="128.27" y2="139.7" width="0.1524" layer="91"/>
+<wire x1="128.27" y1="139.7" x2="119.38" y2="139.7" width="0.1524" layer="91"/>
+<label x="119.38" y="139.7" size="1.778" layer="95" rot="R180" xref="yes"/>
+</segment>
+</net>
+<net name="N$7" class="0">
+<segment>
+<pinref part="D" gate="G$1" pin="P$1"/>
+<wire x1="118.11" y1="132.08" x2="130.81" y2="132.08" width="0.1524" layer="91"/>
+<wire x1="130.81" y1="132.08" x2="130.81" y2="144.78" width="0.1524" layer="91"/>
+<pinref part="U1" gate="G$1" pin="PA13"/>
+<wire x1="130.81" y1="144.78" x2="135.89" y2="144.78" width="0.1524" layer="91"/>
 </segment>
 </net>
@@
 </segment>
 </net>
-<net name="USART1_RTS" class="0">
+<net name="UART1_RTS" class="0">
 <segment>
 <pinref part="U3" gate="G$1" pin="!CTS!"/>
@@
 </segment>
 </net>
-<net name="USART1_CTS" class="0">
+<net name="UART1_CTS" class="0">
 <segment>
 <pinref part="U3" gate="G$1" pin="!RTS!"/>
@@
 </segment>
 </net>
-<net name="USART1_RX" class="0">
+<net name="UART1_RX" class="0">
 <segment>
 <pinref part="U3" gate="G$1" pin="TXD"/>
@@
 </segment>
 </net>
-<net name="USART1_TX" class="0">
+<net name="UART1_TX" class="0">
 <segment>
 <pinref part="U3" gate="G$1" pin="RXD"/>

Commit message: - PCB is done - Generated all output files
Parts:
- removed JP1: (no value), jumper:JP1E
- added J2: 3-644456-2, Hexabitz:3-644456-2
- U2: value LM3940IMP-3.3 -> FT230XQ-R; device Hexabitz:LM3940IMP-3.3 -> Hexabitz:FT230XQ-R
- U3: value FT230XQ-R -> LM3940IMP-3.3; device Hexabitz:FT230XQ-R -> Hexabitz:LM3940IMP-3.3
Connections:
- new net N$8: U3.GND
- net GND: now also U1.PA15, U1.PB1, U1.PB14, U1.PC14-OSC32_IN, U2.GND@13, U2.GND@17, U2.GND@3, U3.GND_2; no longer U2.GND, U2.GND_2, U3.GND@13, U3.GND@17, U3.GND@3
- net N$10: now also J2.2; no longer JP1.2
- net N$11: now also U3.IN; no longer U2.IN
- net N$12: now also U2.USBDP; no longer U3.USBDP
- net N$13: now also U2.USBDM; no longer U3.USBDM
- net N$14: now also U2.CBUS2; no longer U3.CBUS2
- net N$15: now also U2.CBUS1; no longer U3.CBUS1
- net N$18: now also J2.1; no longer JP1.1
- net UART1_CTS: now also U2.!RTS!; no longer U3.!RTS!
- net UART1_RTS: now also U2.!CTS!; no longer U3.!CTS!
- net UART1_RX: now also U2.TXD; no longer U3.TXD
- net UART1_TX: now also U2.RXD; no longer U3.RXD
- net VBUS_SENSE: now also U2.CBUS3; no longer U3.CBUS3
- net VDD: now also U2.!RESET!, U2.3V3OUT, U2.VCC, U2.VCCIO, U3.OUT; no longer U2.OUT, U3.!RESET!, U3.3V3OUT, U3.VCC, U3.VCCIO
