File: H1AR20/Design/H1AR20.sch (EAGLE design)
At the start: 42 parts, among them J1 67503-1020, P1 HEXABIT_17.32_NO_P3, U1 STM32F091CBU6, U2 FT230XQ-R, U3 LM3940IMP-3.3, X1 XTALL_CSTCE8M00G52

Commit message: minor changes in PCB..
Parts:
- renumbered J1 to USB-B*
Changed lines of the file:
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@@
 <part name="SUPPLY1" library="supply2" library_urn="urn:adsk.eagle:library:372" deviceset="VDD" device=""/>
 <part name="SUPPLY2" library="supply2" library_urn="urn:adsk.eagle:library:372" deviceset="GND" device=""/>
-<part name="J1" library="Hexabitz" deviceset="67503-1020" device=""/>
+<part name="USB-B*" library="Hexabitz" deviceset="67503-1020" device=""/>
 <part name="U2" library="Hexabitz" deviceset="FT230XQ-R" device=""/>
 <part name="SUPPLY14" library="supply2" library_urn="urn:adsk.eagle:library:372" deviceset="GND" device=""/>
@@
 </plain>
 <instances>
-<instance part="J1" gate="G$1" x="27.94" y="116.84" smashed="yes">
+<instance part="USB-B*" gate="G$1" x="27.94" y="116.84" smashed="yes">
 <attribute name="NAME" x="27.9578" y="127.00648125" size="1.78026875" layer="95" align="center"/>
 <attribute name="VALUE" x="27.9445" y="104.1367" size="1.77858125" layer="96" align="center"/>
@@
 <segment>
 <pinref part="SUPPLY14" gate="GND" pin="GND"/>
-<pinref part="J1" gate="G$1" pin="GND"/>
+<pinref part="USB-B*" gate="G$1" pin="GND"/>
 <wire x1="43.18" y1="95.25" x2="43.18" y2="109.22" width="0.1524" layer="91"/>
 <wire x1="43.18" y1="109.22" x2="43.18" y2="111.76" width="0.1524" layer="91"/>
 <wire x1="43.18" y1="111.76" x2="39.37" y2="111.76" width="0.1524" layer="91"/>
-<pinref part="J1" gate="G$1" pin="SHEILD"/>
+<pinref part="USB-B*" gate="G$1" pin="SHEILD"/>
 <wire x1="39.37" y1="109.22" x2="43.18" y2="109.22" width="0.1524" layer="91"/>
 <junction x="43.18" y="109.22"/>
@@
 <net name="N$2" class="0">
 <segment>
-<pinref part="J1" gate="G$1" pin="D-"/>
+<pinref part="USB-B*" gate="G$1" pin="D-"/>
 <wire x1="39.37" y1="119.38" x2="92.71" y2="119.38" width="0.1524" layer="91"/>
 <pinref part="C14" gate="G$1" pin="1"/>
@@
 <pinref part="R5" gate="G$1" pin="1"/>
 <wire x1="104.14" y1="114.3" x2="80.01" y2="114.3" width="0.1524" layer="91"/>
-<pinref part="J1" gate="G$1" pin="D+"/>
+<pinref part="USB-B*" gate="G$1" pin="D+"/>
 <wire x1="39.37" y1="116.84" x2="60.96" y2="116.84" width="0.1524" layer="91"/>
 <wire x1="60.96" y1="116.84" x2="60.96" y2="114.3" width="0.1524" layer="91"/>
@@
 <net name="N$18" class="0">
 <segment>
-<pinref part="J1" gate="G$1" pin="VBUS"/>
+<pinref part="USB-B*" gate="G$1" pin="VBUS"/>
 <wire x1="39.37" y1="121.92" x2="50.8" y2="121.92" width="0.1524" layer="91"/>
 <pinref part="R8" gate="G$1" pin="2"/>

Commit message: replaced (USB-B*) with (PUSB*) and fixed gerber files
Parts:
- renumbered USB-B* to PUSB*
Changed lines of the file:
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@@
 <part name="SUPPLY1" library="supply2" library_urn="urn:adsk.eagle:library:372" deviceset="VDD" device=""/>
 <part name="SUPPLY2" library="supply2" library_urn="urn:adsk.eagle:library:372" deviceset="GND" device=""/>
-<part name="USB-B*" library="Hexabitz" deviceset="67503-1020" device=""/>
+<part name="PUSB*" library="Hexabitz" deviceset="67503-1020" device=""/>
 <part name="U2" library="Hexabitz" deviceset="FT230XQ-R" device=""/>
 <part name="SUPPLY14" library="supply2" library_urn="urn:adsk.eagle:library:372" deviceset="GND" device=""/>
@@
 </plain>
 <instances>
-<instance part="USB-B*" gate="G$1" x="27.94" y="116.84" smashed="yes">
+<instance part="PUSB*" gate="G$1" x="27.94" y="116.84" smashed="yes">
 <attribute name="NAME" x="27.9578" y="127.00648125" size="1.78026875" layer="95" align="center"/>
 <attribute name="VALUE" x="27.9445" y="104.1367" size="1.77858125" layer="96" align="center"/>
@@
 <segment>
 <pinref part="SUPPLY14" gate="GND" pin="GND"/>
-<pinref part="USB-B*" gate="G$1" pin="GND"/>
+<pinref part="PUSB*" gate="G$1" pin="GND"/>
 <wire x1="43.18" y1="95.25" x2="43.18" y2="109.22" width="0.1524" layer="91"/>
 <wire x1="43.18" y1="109.22" x2="43.18" y2="111.76" width="0.1524" layer="91"/>
 <wire x1="43.18" y1="111.76" x2="39.37" y2="111.76" width="0.1524" layer="91"/>
-<pinref part="USB-B*" gate="G$1" pin="SHEILD"/>
+<pinref part="PUSB*" gate="G$1" pin="SHEILD"/>
 <wire x1="39.37" y1="109.22" x2="43.18" y2="109.22" width="0.1524" layer="91"/>
 <junction x="43.18" y="109.22"/>
@@
 <net name="N$2" class="0">
 <segment>
-<pinref part="USB-B*" gate="G$1" pin="D-"/>
+<pinref part="PUSB*" gate="G$1" pin="D-"/>
 <wire x1="39.37" y1="119.38" x2="92.71" y2="119.38" width="0.1524" layer="91"/>
 <pinref part="C14" gate="G$1" pin="1"/>
@@
 <pinref part="R5" gate="G$1" pin="1"/>
 <wire x1="104.14" y1="114.3" x2="80.01" y2="114.3" width="0.1524" layer="91"/>
-<pinref part="USB-B*" gate="G$1" pin="D+"/>
+<pinref part="PUSB*" gate="G$1" pin="D+"/>
 <wire x1="39.37" y1="116.84" x2="60.96" y2="116.84" width="0.1524" layer="91"/>
 <wire x1="60.96" y1="116.84" x2="60.96" y2="114.3" width="0.1524" layer="91"/>
@@
 <net name="N$18" class="0">
 <segment>
-<pinref part="USB-B*" gate="G$1" pin="VBUS"/>
+<pinref part="PUSB*" gate="G$1" pin="VBUS"/>
 <wire x1="39.37" y1="121.92" x2="50.8" y2="121.92" width="0.1524" layer="91"/>
 <pinref part="R8" gate="G$1" pin="2"/>
