File: H1AR20/Design/H1AR20.brd (EAGLE design)
At the start: 34.6 x 30 mm, 42 parts, among them J1 67503-1020, P1 HEXABIT_17.32_NO_P3, U1 STM32F091CBU6, U2 FT230XQ-R, U3 LM3940IMP-3.3, X1 XTALL_CSTCE8M00G52

Commit message: minor changes in PCB..
Parts:
- renumbered J1 to USB-B*

Commit message: replaced (USB-B*) with (PUSB*) and fixed gerber files
Parts:
- renumbered USB-B* to PUSB*
Changed lines of the file:
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@@
 </element>
 <element name="P1" library="hexabitz_connectors" package="HEXABIT_17.32_NO_P3" value="HEXABIT_17.32_NO_P3" x="34.6202" y="34.6202" smashed="yes"/>
-<element name="USB-B*" library="Hexabitz" package="67503-1020" value="67503-1020" x="34.2646" y="19.685" smashed="yes" rot="R90">
+<element name="PUSB*" library="Hexabitz" package="67503-1020" value="67503-1020" x="34.2646" y="19.685" smashed="yes" rot="R90">
 <attribute name="DESCRIPTION" value=" USB - mini B USB 2.0 OTG Receptacle Connector 5 Position Surface Mount, Right Angle " x="34.2646" y="19.685" size="1.778" layer="27" rot="R90" display="off"/>
 <attribute name="MFN" value="Molex" x="34.2646" y="19.685" size="1.778" layer="27" rot="R90" display="off"/>
@@
 <contactref element="U2" pad="13"/>
 <contactref element="U2" pad="17"/>
-<contactref element="USB-B*" pad="5"/>
-<contactref element="USB-B*" pad="9"/>
-<contactref element="USB-B*" pad="10"/>
-<contactref element="USB-B*" pad="11"/>
-<contactref element="USB-B*" pad="8"/>
+<contactref element="PUSB*" pad="5"/>
+<contactref element="PUSB*" pad="9"/>
+<contactref element="PUSB*" pad="10"/>
+<contactref element="PUSB*" pad="11"/>
+<contactref element="PUSB*" pad="8"/>
 <contactref element="C17" pad="2"/>
 <contactref element="C16" pad="1"/>
@@
 </signal>
 <signal name="N$2">
-<contactref element="USB-B*" pad="2"/>
+<contactref element="PUSB*" pad="2"/>
 <contactref element="C14" pad="1"/>
 <contactref element="R4" pad="1"/>
@@
 <contactref element="C13" pad="1"/>
 <contactref element="R5" pad="1"/>
-<contactref element="USB-B*" pad="3"/>
+<contactref element="PUSB*" pad="3"/>
 <wire x1="38.8375" y1="23.2029" x2="37.8088" y2="23.2029" width="0.254" layer="16"/>
 <wire x1="37.8088" y1="23.2029" x2="36.9824" y2="22.3765" width="0.254" layer="16"/>
@@
 </signal>
 <signal name="N$18">
-<contactref element="USB-B*" pad="1"/>
+<contactref element="PUSB*" pad="1"/>
 <contactref element="R8" pad="2"/>
 <contactref element="PWR" pad="1"/>
